File: B+ Delay/B+ Delay.kicad_pcb (KiCad board)
At the start: 2 copper layers, 80 x 68 mm, 31 parts, among them J1 Pwr in, J2 B+ IN, J3 B+ Out, J4 LED, Q3 MMBT3904, Q4 MMBT3906, U1 LM7805_TO220, U2 SE556, U3 CPC1779

Commit message: Add files via upload
Parts:
- added U4: CPC1779, CH parts:CPC1779J, F.Cu at (177.9, -336.1)
- moved J3 57.6 mm to (156.0, -332.4), turned to 90 degrees
- moved J2 27.0 mm to (156.0, -319.4), turned to 90 degrees
- moved U3 17.4 mm to (175.9, -326.6)
- moved J1 10.6 mm to (155.8, -308.8)
- moved D6 8.08 mm to (167.0, -310.7)
- moved R1 8.08 mm to (199.5, -320.7)
- moved U1 8.08 mm to (194.5, -313.4)
- moved C6 8.08 mm to (181.5, -312.9)
- moved C9 8.08 mm to (208.5, -312.4)
- moved Q3 4.51 mm to (162.6, -302.1)
Connections:
- J3 pad 2: Net-(J2-Pin_2) -> Net-(J3-Pin_2)
Routing:
- net Net-(J3-Pin_2): track 0.00 -> 33.8 mm
- net Net-(J2-Pin_2): track 50.9 -> 27.2 mm
- net Net-(Q3-C): track 89.4 -> 79.1 mm
- net GND: track 48.2 -> 41.1 mm, vias 10 -> 9
- net Net-(R1-Pad2): track 15.3 -> 20.2 mm
- net Net-(Q3-B): track 15.2 -> 10.8 mm
- net Net-(J3-Pin_1): track 26.0 -> 29.7 mm
- net Net-(J2-Pin_1): track 26.0 -> 23.4 mm
- net Net-(J1-Pin_1): track 7.00 -> 9.51 mm
- net +5V: track 109.8 -> 107.9 mm
- net Net-(J1-Pin_2): track 7.02 -> 7.71 mm

Commit message: New rev, dual relay, fixed stuff
Fixing missing ground trace, correct footprint for diode, added test points, changed B++ input/output on terminal block
Parts:
- added JP1: ~, Jumper:SolderJumper-2_P1.3mm_Bridged_RoundedPad1.0x1.5mm, F.Cu at (161.8, -286.0)
- added JP2: ~, Jumper:SolderJumper-2_P1.3mm_Open_RoundedPad1.0x1.5mm, F.Cu at (158.5, -291.5)
- added TP+5: ~, TestPoint:TestPoint_Keystone_5010-5014_Multipurpose, F.Cu at (198.0, -301.0)
- added TP-Delay2: ~, TestPoint:TestPoint_Keystone_5010-5014_Multipurpose, F.Cu at (154.5, -295.5)
- added TP-GND1: ~, TestPoint:TestPoint_Keystone_5010-5014_Multipurpose, F.Cu at (204.0, -301.0)
- added TP-LED1: ~, TestPoint:TestPoint_Keystone_5010-5014_Multipurpose, F.Cu at (214.0, -289.0)
- added TP-Relay1: ~, TestPoint:TestPoint_Keystone_5010-5014_Multipurpose, F.Cu at (195.0, -342.5)
- added TP-Relay2: ~, TestPoint:TestPoint_Keystone_5010-5014_Multipurpose, F.Cu at (188.5, -342.5)
- added TP-voltageDiv1: ~, TestPoint:TestPoint_Keystone_5010-5014_Multipurpose, F.Cu at (167.0, -302.0)
- D5: footprint Diode_SMD:D_0805_2012Metric_Pad1.15x1.40mm_HandSolder -> Diode_SMD:D_SOD-123
- J2: value B+ IN -> B+ A
- J3: value B+ Out -> B+ B
- moved D5 0.25 mm to (163.0, -289.0)
Connections:
- J2 pad 2: Net-(J2-Pin_2) -> A
- J3 pad 1: Net-(J3-Pin_1) -> B
- U2 pad 4: Net-(D5-K) -> Net-(JP1-B)
- U3 pad 2: Net-(J3-Pin_1) -> A
- U4 pad 1: Net-(J2-Pin_2) -> B
Routing:
- net Net-(J3-Pin_1): track 29.7 -> 0.00 mm
- net A: track 0.00 -> 29.2 mm
- net Net-(J2-Pin_2): track 27.2 -> 0.00 mm
- net B: track 0.00 -> 23.4 mm
- net Net-(JP1-B): track 0.00 -> 20.3 mm
- net +5V: track 107.9 -> 123.1 mm
- net Net-(Q4-C): track 4.19 -> 11.4 mm
- net Net-(R1-Pad2): track 20.2 -> 27.3 mm
- net Net-(Q3-C): track 79.1 -> 85.8 mm
- net GND: track 41.1 -> 45.7 mm, vias 9 -> 10
- net Net-(U2A-Q): track 10.0 -> 14.3 mm, vias 0 -> 2
- net Net-(Q3-B): track 10.8 -> 14.7 mm
- net Net-(D5-K): track 16.0 -> 13.7 mm
- net Net-(J2-Pin_1): track 23.4 -> 25.5 mm
Other:
- board text added: "Millett/Heisey B++ Delay Rev 4"
